File: hardware/din-synch-hub.sch (EAGLE design)
At the start: 47 parts, among them IC1 6N138, IC2 PIC12F1822SO08, IC3 4050D, IC4 REG1117, IC6 4050D, X1 DIN5PIN, X2 DIN5PIN, X3 DIN5PIN, X4 DIN5PIN, X5 DIN5PIN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

Commit message: updates
Parts:
- C3: device rcl:C-EUC0805 -> rcl:CPOL-EUE2,5-6E
- C7: device rcl:CPOL-EUE2,5-6E -> rcl:C-EUC0805
Connections:
- net GND: now also C3.-, C5.2, C7.1, R3.2, R4.1; no longer C3.2, C5.1, C7.-, R14.2, R16.1
- net IN: now also R1.1; no longer R15.1
- net N$1: now also R6.1; no longer R1.1
- net N$10: now also R10.2; no longer R5.2
- net N$11: now also R9.2; no longer R6.2
- net N$12: now also R9.1; no longer R6.1
- net N$13: now also R12.1; no longer R7.1
- net N$14: now also R12.2; no longer R7.2
- net N$15: now also R11.1; no longer R8.1
- net N$16: now also R11.2; no longer R8.2
- net N$17: now also R14.1; no longer R9.1
- net N$18: now also R14.2; no longer R9.2
- net N$19: now also R13.1; no longer R10.1
- net N$2: now also R6.2; no longer R1.2
- net N$20: now also R13.2; no longer R10.2
- net N$21: now also R16.1; no longer R11.1
- net N$22: now also R16.2; no longer R11.2
- net N$23: now also R15.2; no longer R12.2
- net N$24: now also R15.1; no longer R12.1
- net N$26: now also R2.1; no longer R13.1
- net N$27: now also R2.2; no longer R13.2
- net N$29: now also R3.1; no longer R14.1
- net N$3: now also R5.1; no longer R2.1
- net N$30: now also R4.2; no longer R16.2
- net N$32: now also C3.+; no longer C6.+
- net N$4: now also R5.2; no longer R2.2
- net N$5: now also R8.1; no longer R3.1
- net N$6: now also R8.2; no longer R3.2
- net N$7: now also R7.1; no longer R4.1
- net N$8: now also R7.2; no longer R4.2
- net N$9: now also R10.1; no longer R5.1
- net VCC: now also C5.1, C6.+, C7.2, R1.2; no longer C3.1, C5.2, C7.+, R15.2
Other:
- moved on the sheet: C1, C2, C5, C6, R1, R10, R11, R12, R13, R14, R15, R16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
